File: hardware/pcb/greenhouse-controller.kicad_sch (KiCad schematic)
At the start: 69 parts, among them J1 Motor 2, J10 ALARM contact, J11 AC-Mains, J12 DM1AA-SF-PEJ72, J2 24V in, J3 I2C Display, J4 Keypad, J5 MODBUS RS485 S200, J6 Motor 3, J7 Motor 1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

Commit message: intermediate update PCB
Parts:
- added J8: Load enable, Connector_PinHeader_2.54mm:PinHeader_1x02_P2.54mm_Vertical, symbol Connector_Generic:Conn_01x02
Connections:
- net RS485-B: now also J8.1 (Pin_1); no longer R21.2
- new net: J8.2 (Pin_2), R21.2
Other:
- moved on the sheet: D13, R21
Changed lines of the file:
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@@
 	)
 	(junction
-		(at 210.82 190.5)
+		(at 257.81 129.54)
 		(diameter 0)
 		(color 0 0 0 0)
 	)
 	(junction
-		(at 326.39 60.96)
+		(at 210.82 190.5)
 		(diameter 0)
 		(color 0 0 0 0)
 	)
 	(junction
-		(at 246.38 25.4)
+		(at 326.39 60.96)
 		(diameter 0)
 		(color 0 0 0 0)
 	)
 	(junction
-		(at 248.92 129.54)
+		(at 246.38 25.4)
 		(diameter 0)
 		(color 0 0 0 0)
@@
 	)
 	(junction
-		(at 231.14 125.73)
-		(diameter 0)
-		(color 0 0 0 0)
-	)
-	(junction
 		(at 246.38 60.96)
 		(diameter 0)
@@
 	)
 	(junction
-		(at 240.03 133.35)
+		(at 326.39 173.99)
 		(diameter 0)
 		(color 0 0 0 0)
 	)
 	(junction
-		(at 326.39 173.99)
+		(at 231.14 129.54)
 		(diameter 0)
 		(color 0 0 0 0)
@@
 	)
 	(junction
+		(at 248.92 133.35)
+		(diameter 0)
+		(color 0 0 0 0)
+	)
+	(junction
 		(at 73.66 223.52)
 		(diameter 0)
@@
 	)
 	(junction
+		(at 240.03 125.73)
+		(diameter 0)
+		(color 0 0 0 0)
+	)
+	(junction
 		(at 339.09 153.67)
 		(diameter 0)
@@
 	)
 	(junction
-		(at 219.71 129.54)
-		(diameter 0)
-		(color 0 0 0 0)
-	)
-	(junction
 		(at 339.09 120.65)
 		(diameter 0)
@@
 	(wire
 		(pts
-			(xy 240.03 133.35) (xy 271.78 133.35)
-		)
-		(stroke
-			(width 0)
-			(type default)
-		)
-	)
-	(wire
-		(pts
 			(xy 40.64 165.1) (xy 64.77 165.1)
 		)
@@
 	(wire
 		(pts
+			(xy 248.92 133.35) (xy 271.78 133.35)
+		)
+		(stroke
+			(width 0)
+			(type default)
+		)
+	)
+	(wire
+		(pts
 			(xy 40.64 125.73) (xy 66.04 125.73)
 		)
@@
 	(wire
 		(pts
+			(xy 257.81 129.54) (xy 271.78 129.54)
+		)
+		(stroke
+			(width 0)
+			(type default)
+		)
+	)
+	(wire
+		(pts
 			(xy 133.35 74.93) (xy 154.94 74.93)
 		)
@@
 	(wire
 		(pts
-			(xy 217.17 125.73) (xy 231.14 125.73)
+			(xy 217.17 125.73) (xy 240.03 125.73)
 		)
 		(stroke
@@
 	(wire
 		(pts
+			(xy 240.03 125.73) (xy 240.03 140.97)
+		)
+		(stroke
+			(width 0)
+			(type default)
+		)
+	)
+	(wire
+		(pts
 			(xy 66.04 205.74) (xy 86.36 205.74)
 		)
@@
 	(wire
 		(pts
-			(xy 231.14 125.73) (xy 231.14 140.97)
-		)
-		(stroke
-			(width 0)
-			(type default)
-		)
-	)
-	(wire
-		(pts
 			(xy 66.04 231.14) (xy 86.36 231.14)
 		)
@@
 	(wire
 		(pts
-			(xy 219.71 129.54) (xy 248.92 129.54)
-		)
-		(stroke
-			(width 0)
-			(type default)
-		)
-	)
-	(wire
-		(pts
 			(xy 311.15 173.99) (xy 326.39 173.99)
 		)
@@
 	(wire
 		(pts
-			(xy 231.14 125.73) (xy 271.78 125.73)
-		)
-		(stroke
-			(width 0)
-			(type default)
-		)
-	)
-	(wire
-		(pts
 			(xy 144.78 125.73) (xy 160.02 125.73)
 		)
@@
 	(wire
 		(pts
-			(xy 248.92 129.54) (xy 248.92 140.97)
+			(xy 257.81 129.54) (xy 257.81 140.97)
 		)
 		(stroke
@@
 	(wire
 		(pts
+			(xy 240.03 125.73) (xy 271.78 125.73)
+		)
+		(stroke
+			(width 0)
+			(type default)
+		)
+	)
+	(wire
+		(pts
 			(xy 339.09 76.2) (xy 345.44 76.2)
 		)
@@
 	(wire
 		(pts
-			(xy 205.74 129.54) (xy 219.71 129.54)
+			(xy 205.74 129.54) (xy 231.14 129.54)
 		)
 		(stroke
@@
 	(wire
 		(pts
-			(xy 248.92 129.54) (xy 271.78 129.54)
+			(xy 339.09 60.96) (xy 339.09 63.5)
 		)
 		(stroke
@@
 	(wire
 		(pts
-			(xy 339.09 60.96) (xy 339.09 63.5)
+			(xy 177.8 271.78) (xy 210.82 271.78)
 		)
 		(stroke
@@
 	(wire
 		(pts
-			(xy 177.8 271.78) (xy 210.82 271.78)
+			(xy 66.04 198.12) (xy 86.36 198.12)
 		)
 		(stroke
@@
 	(wire
 		(pts
-			(xy 66.04 198.12) (xy 86.36 198.12)
+			(xy 81.28 49.53) (xy 102.87 49.53)
 		)
 		(stroke
@@
 	(wire
 		(pts
-			(xy 81.28 49.53) (xy 102.87 49.53)
+			(xy 326.39 105.41) (xy 311.15 105.41)
 		)
 		(stroke
@@
 	(wire
 		(pts
-			(xy 326.39 105.41) (xy 311.15 105.41)
+			(xy 220.98 146.05) (xy 217.17 146.05)
 		)
 		(stroke
@@
 	(wire
 		(pts
-			(xy 219.71 129.54) (xy 219.71 135.89)
+			(xy 231.14 129.54) (xy 231.14 135.89)
 		)
 		(stroke
@@
 	(wire
 		(pts
-			(xy 219.71 143.51) (xy 219.71 146.05)
+			(xy 231.14 143.51) (xy 231.14 146.05)
 		)
 		(stroke
@@
 	(wire
 		(pts
-			(xy 205.74 133.35) (xy 240.03 133.35)
+			(xy 205.74 133.35) (xy 248.92 133.35)
 		)
 		(stroke
@@
 	(wire
 		(pts
+			(xy 231.14 129.54) (xy 257.81 129.54)
+		)
+		(stroke
+			(width 0)
+			(type default)
+		)
+	)
+	(wire
+		(pts
 			(xy 74.93 219.71) (xy 73.66 219.71)
 		)
@@
 	(wire
 		(pts
-			(xy 219.71 146.05) (xy 217.17 146.05)
+			(xy 231.14 146.05) (xy 223.52 146.05)
 		)
 		(stroke
@@
 	(wire
 		(pts
-			(xy 240.03 133.35) (xy 240.03 137.16)
+			(xy 248.92 133.35) (xy 248.92 137.16)
 		)
 		(stroke
@@
 	(symbol
 		(lib_id "Diode:SM712_SOT23")
-		(at 240.03 140.97 180)
+		(at 248.92 140.97 180)
 		(unit 1)
 		(exclude_from_sim no)
@@
 		(fields_autoplaced yes)
 		(property "Reference" "D13"
-			(at 240.03 144.78 0)
+			(at 248.92 144.78 0)
 			(effects
 				(font
@@
 		)
 		(property "Value" "SM712_SOT23"
-			(at 240.03 147.32 0)
+			(at 248.92 147.32 0)
 			(effects
 				(font
@@
 		)
 		(property "Footprint" "Package_TO_SOT_SMD:SOT-23"
-			(at 240.03 132.08 0)
+			(at 248.92 132.08 0)
 			(effects
 				(font
@@
 		)
 		(property "Datasheet" "https://www.littelfuse.com/~/media/electronics/datasheets/tvs_diode_arrays/littelfuse_tvs_diode_array_sm712_datasheet.pdf.pdf"
-			(at 243.84 140.97 0)
+			(at 252.73 140.97 0)
 			(effects
 				(font
@@
 		)
 		(property "Description" "7V/12V, 600W Asymmetrical TVS Diode Array, SOT-23"
-			(at 240.03 140.97 0)
+			(at 248.92 140.97 0)
 			(effects
 				(font
@@
 	)
 	(symbol
+		(lib_id "Connector_Generic:Conn_01x02")
+		(at 220.98 140.97 90)
+		(unit 1)
+		(exclude_from_sim no)
+		(in_bom yes)
+		(on_board yes)
+		(dnp no)
+		(property "Reference" "J8"
+			(at 226.06 139.6999 90)
+			(effects
+				(font
+					(size 1.27 1.27)
+				)
+				(justify right)
+			)
+		)
+		(property "Value" "Load enable"
+			(at 216.662 148.082 90)
+			(effects
+				(font
+					(size 1.27 1.27)
+				)
+				(justify right)
+			)
+		)
+		(property "Footprint" "Connector_PinHeader_2.54mm:PinHeader_1x02_P2.54mm_Vertical"
+			(at 220.98 140.97 0)
+			(effects
+				(font
+					(size 1.27 1.27)
+				)
+				(hide yes)
+			)
+		)
+		(property "Datasheet" "~"
+			(at 220.98 140.97 0)
+			(effects
+				(font
+					(size 1.27 1.27)
+				)
+				(hide yes)
+			)
+		)
+		(property "Description" "Generic connector, single row, 01x02, script generated (kicad-library-utils/schlib/autogen/connector/)"
+			(at 220.98 140.97 0)
+			(effects
+				(font
+					(size 1.27 1.27)
+				)
+				(hide yes)
+			)
+		)
+		(pin "2"
+		)
+		(pin "1"
+		)
+		(instances
+			(project ""
+				(path "/2be5eb1b-bfdc-4766-9909-5178f7452cd9"
+					(reference "J8")
+					(unit 1)
+				)
+			)
+		)
+	)
+	(symbol
 		(lib_id "Transistor_FET:2N7000")
 		(at 336.55 82.55 0)
@@
 	(symbol
 		(lib_id "Device:R")
-		(at 219.71 139.7 0)
+		(at 231.14 139.7 0)
 		(unit 1)
 		(exclude_from_sim no)
@@
 		(fields_autoplaced yes)
 		(property "Reference" "R21"
-			(at 222.25 138.4299 0)
+			(at 233.68 138.4299 0)
 			(effects
 				(font
@@
 		)
 		(property "Value" "120"
-			(at 222.25 140.9699 0)
+			(at 233.68 140.9699 0)
 			(effects
 				(font
@@
 		)
 		(property "Footprint" "Resistor_SMD:R_1206_3216Metric_Pad1.30x1.75mm_HandSolder"
-			(at 217.932 139.7 90)
+			(at 229.362 139.7 90)
 			(effects
 				(font
@@
 		)
 		(property "Datasheet" "~"
-			(at 219.71 139.7 0)
+			(at 231.14 139.7 0)
 			(effects
 				(font
@@
 		)
 		(property "Description" "Resistor"
-			(at 219.71 139.7 0)
+			(at 231.14 139.7 0)
 			(effects
 				(font

Commit message: Added RGB-led feature for controller state, added documentation for S200 wind sensor
Connections:
- net 3V3: no longer C4.1, U4.8 (VCC)
- net 5V: now also C4.1, U4.8 (VCC)
Changed lines of the file:
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@@
 		)
 	)
-	(label "3V3"
+	(label "5V"
 		(at 179.07 158.75 0)
 		(effects
