File: hardware/pcb/greenhouse-controller.kicad_sch (KiCad schematic)
At the start: 70 parts, among them J1 Motor 2, J10 ALARM contact, J11 AC-Mains, J12 DM1AA-SF-PEJ72, J2 24V in, J3 I2C Display, J4 Keypad, J5 MODBUS RS485 S200, J6 Motor 3, J7 Motor 1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

Commit message: PCB bump to V1.1.0
Parts:
- removed J5: MODBUS RS485 S200, TerminalBlock_Phoenix:TerminalBlock_Phoenix_MKDS-1,5-8_1x08_P5.00mm_Horizontal, symbol Connector:Screw_Terminal_01x08
- added J13: MODBUS RS485 S200, TerminalBlock_Phoenix:TerminalBlock_Phoenix_MKDS-1,5-4_1x04_P5.00mm_Horizontal, symbol Connector:Screw_Terminal_01x04
Connections:
- net 24V: now also J13.1 (Pin_1)
- net GND: now also J13.2 (Pin_2)
- net RS485-A: now also J13.3 (Pin_3)
- net RS485-B: now also J13.4 (Pin_4)
Other:
- moved on the sheet: J9
